Commit message: feat: Clone udacity_bot to  xbot
Add xbot as udacity_bot to modify

File: udacity_bot/urdf/udacity_bot.xacro (robot description, xacro)
@@ -36,5 +36,5 @@
   </link>
   <joint type="fixed" name="hokuyo_joint">
-    <origin xyz="0.15 0 0.1" rpy="0 0 0"/>
+    <origin xyz="0.15 0 0.085" rpy="0 0 0"/>
     <child link="hokuyo"/>
     <parent link="chassis"/>
@@ -135,5 +135,5 @@
       />
     </inertial>
-    <collision name='chassis_collision'>
+    <collision name='collision'>
       <origin xyz="0 0 0" rpy=" 0 0 0"/>
       <geometry>
