Commit message: feat: Add sensor_base link
Add sensor_base link to modify the sensor locations.

File: xbot/urdf/xbot.xacro (robot description, xacro)
@@ -9,7 +9,7 @@
   </joint>
   <joint type="fixed" name="camera_joint">
-    <origin xyz="0.2 0 0" rpy="0 0 0"/>
+    <origin xyz="0.175 0 0" rpy="0 0 0"/>
     <child link="camera"/>
-    <parent link="chassis"/>
+    <parent link="sensor_base"/>
   </joint>
  <link name='camera'>
@@ -36,7 +36,7 @@
   </link>
   <joint type="fixed" name="hokuyo_joint">
-    <origin xyz="0.15 0 0.085" rpy="0 0 0"/>
+    <origin xyz="0.0 0 0.05" rpy="0 0 0"/>
     <child link="hokuyo"/>
-    <parent link="chassis"/>
+    <parent link="sensor_base"/>
   </joint>
  <link name='hokuyo'>
@@ -63,5 +63,5 @@
   </link>
   <joint type="continuous" name="left_wheel_hinge">
-    <origin xyz="0 0.15 0" rpy="0 0 0"/>
+    <origin xyz="0.0 0.15 0" rpy="0 0 0"/>
     <child link="left_wheel"/>
     <parent link="chassis"/>
@@ -94,5 +94,5 @@
   </link>
   <joint type="continuous" name="right_wheel_hinge">
-    <origin xyz="0 -0.15 0" rpy="0 0 0"/>
+    <origin xyz="0.0 -0.15 0" rpy="0 0 0"/>
     <child link="right_wheel"/>
     <parent link="chassis"/>
@@ -124,4 +124,33 @@
     </visual>
   </link>
+  <joint type="fixed" name="sensor_base_joint">
+    <origin xyz="0.0 0.0 0.075" rpy="0 0 0"/>
+    <child link="sensor_base"/>
+    <parent link="chassis"/>
+  </joint>
+  <link name='sensor_base'>
+    <pose>0 0 0.1 0 0 0</pose>
+    <inertial>
+      <mass value="1.40625"/>
+      <origin xyz="0 0 0" rpy="0 0 0"/>
+      <inertia
+          ixx="0.1" ixy="0" ixz="0"
+          iyy="0.1" iyz="0"
+          izz="0.1"
+      />
+    </inertial>
+    <collision name='sensor_base_collision'>
+      <origin xyz="0 0 0" rpy=" 0 0 0"/>
+      <geometry>
+        <box size=".3 .05 .05"/>
+      </geometry>
+    </collision>
+    <visual name='sensor_base_visual'>
+      <origin xyz="0 0 0" rpy=" 0 0 0"/>
+      <geometry>
+        <box size=".3 .05 .05"/>
+      </geometry>
+    </visual>
+  </link>
   <link name='chassis'>
     <pose>0 0 0.1 0 0 0</pose>
@@ -160,4 +189,5 @@
     </visual>
     <collision name='front_caster_collision'>
+      <material>Gazebo/Red</material>
       <origin xyz="0.15 0 -0.05" rpy=" 0 0 0"/>
       <geometry>
